File: Usb_a-to-pinhead.kicad_sch (KiCad schematic)
At the start: 4 parts, among them J1 USB_A, J2 Conn_01x02_Pin

Commit message: 2026-03-9 | So-Mo
Parts:
- added C1: 100nF, Capacitor_SMD:C_0402_1005Metric, symbol Device:C
Connections:
- net +5V: now also C1.1
- net GND: now also C1.2
Other:
- note added: "Additional"
- note added: "USB_to_pinhead"
- moved on the sheet: D1, J1, J2, R1
